File: Hardware/OLED Display.sch (EAGLE design)
At the start: 30 parts, among them J1 QWIIC_RIGHT_ANGLE, J3 QWIIC_RIGHT_ANGLE, U2 APX803S-SA, U3 AMO091-12832BFG02-H14

Commit message: Swaps right angle Qwiic connector to vertical
Parts:
- J1, J3: value QWIIC_RIGHT_ANGLE -> Vertical Qwiic Connector; device SparkFun-Connectors:QWIIC_CONNECTORJS-1MM -> SparkFun-Connectors:QWIIC_CONNECTOR
Changed lines of the file:
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@@
 <part name="SUPPLY4" library="SparkFun-PowerSymbols" deviceset="3.3V" device=""/>
 <part name="SUPPLY5" library="SparkFun-PowerSymbols" deviceset="3.3V" device=""/>
-<part name="J3" library="SparkFun-Connectors" deviceset="QWIIC_CONNECTOR" device="JS-1MM" value="QWIIC_RIGHT_ANGLE"/>
-<part name="J1" library="SparkFun-Connectors" deviceset="QWIIC_CONNECTOR" device="JS-1MM" value="QWIIC_RIGHT_ANGLE"/>
+<part name="J3" library="SparkFun-Connectors" deviceset="QWIIC_CONNECTOR" device="" value="Vertical Qwiic Connector"/>
+<part name="J1" library="SparkFun-Connectors" deviceset="QWIIC_CONNECTOR" device="" value="Vertical Qwiic Connector"/>
 <part name="R4" library="SparkFun-Resistors" deviceset="10KOHM" device="-0603-1/10W-1%" value="10k"/>
 <part name="LOGO4" library="SparkFun-Aesthetics" deviceset="SPECIAL_INSTRUCTIONS" device="-ORDERING"/>
@@
 </instance>
 <instance part="J3" gate="J1" x="175.26" y="137.16" smashed="yes" rot="MR0">
-<attribute name="VALUE" x="198.12" y="131.826" size="1.778" layer="96" font="vector" rot="MR0" align="top-left"/>
+<attribute name="VALUE" x="205.74" y="131.826" size="1.778" layer="96" font="vector" rot="MR0" align="top-left"/>
 <attribute name="NAME" x="180.34" y="145.034" size="1.778" layer="95" font="vector" rot="MR0"/>
 </instance>
 <instance part="J1" gate="J1" x="218.44" y="137.16" smashed="yes" rot="MR0">
-<attribute name="VALUE" x="238.76" y="131.826" size="1.778" layer="96" font="vector" rot="MR0" align="top-left"/>
+<attribute name="VALUE" x="248.92" y="131.826" size="1.778" layer="96" font="vector" rot="MR0" align="top-left"/>
 <attribute name="NAME" x="223.52" y="145.034" size="1.778" layer="95" font="vector" rot="MR0"/>
 </instance>
