File: Production/OLED Display-Panel.brd (EAGLE design)
At the start: 199.2 x 132.7 mm, 1158 parts, among them J1 QWIIC_RIGHT_ANGLE, J10 QWIIC_RIGHT_ANGLE, J11 QWIIC_RIGHT_ANGLE, J12 QWIIC_RIGHT_ANGLE, J13 QWIIC_RIGHT_ANGLE, J14 QWIIC_RIGHT_ANGLE, J15 QWIIC_RIGHT_ANGLE, J16 QWIIC_RIGHT_ANGLE, J17 QWIIC_RIGHT_ANGLE, J18 QWIIC_RIGHT_ANGLE, J19 QWIIC_RIGHT_ANGLE, J2 QWIIC_RIGHT_ANGLE, J20 QWIIC_RIGHT_ANGLE, J21 QWIIC_RIGHT_ANGLE, J22 QWIIC_RIGHT_ANGLE, J23 QWIIC_RIGHT_ANGLE, J24 QWIIC_RIGHT_ANGLE, J25 QWIIC_RIGHT_ANGLE, J26 QWIIC_RIGHT_ANGLE, J27 QWIIC_RIGHT_ANGLE, J28 QWIIC_RIGHT_ANGLE, J29 QWIIC_RIGHT_ANGLE, J3 QWIIC_RIGHT_ANGLE, J30 QWIIC_RIGHT_ANGLE, J31 QWIIC_RIGHT_ANGLE, J32 QWIIC_RIGHT_ANGLE, J33 QWIIC_RIGHT_ANGLE, J34 QWIIC_RIGHT_ANGLE, J35 QWIIC_RIGHT_ANGLE, J36 QWIIC_RIGHT_ANGLE, J37 QWIIC_RIGHT_ANGLE, J38 QWIIC_RIGHT_ANGLE, J39 QWIIC_RIGHT_ANGLE, J4 QWIIC_RIGHT_ANGLE, J40 QWIIC_RIGHT_ANGLE, J41 QWIIC_RIGHT_ANGLE, J42 QWIIC_RIGHT_ANGLE, J43 QWIIC_RIGHT_ANGLE, J44 QWIIC_RIGHT_ANGLE, J45 QWIIC_RIGHT_ANGLE, J46 QWIIC_RIGHT_ANGLE, J47 QWIIC_RIGHT_ANGLE, J48 QWIIC_RIGHT_ANGLE, J49 QWIIC_RIGHT_ANGLE, J5 QWIIC_RIGHT_ANGLE, J50 QWIIC_RIGHT_ANGLE, J51 QWIIC_RIGHT_ANGLE, J52 QWIIC_RIGHT_ANGLE, J53 QWIIC_RIGHT_ANGLE, J54 QWIIC_RIGHT_ANGLE, J55 QWIIC_RIGHT_ANGLE, J56 QWIIC_RIGHT_ANGLE, J57 QWIIC_RIGHT_ANGLE, J58 QWIIC_RIGHT_ANGLE, J59 QWIIC_RIGHT_ANGLE, J6 QWIIC_RIGHT_ANGLE, J60 QWIIC_RIGHT_ANGLE, J61 QWIIC_RIGHT_ANGLE, J62 QWIIC_RIGHT_ANGLE, J63 QWIIC_RIGHT_ANGLE, J64 QWIIC_RIGHT_ANGLE, J65 QWIIC_RIGHT_ANGLE, J66 QWIIC_RIGHT_ANGLE, J67 QWIIC_RIGHT_ANGLE, J68 QWIIC_RIGHT_ANGLE, J69 QWIIC_RIGHT_ANGLE, J7 QWIIC_RIGHT_ANGLE, J70 QWIIC_RIGHT_ANGLE, J71 QWIIC_RIGHT_ANGLE, J72 QWIIC_RIGHT_ANGLE, J8 QWIIC_RIGHT_ANGLE, J9 QWIIC_RIGHT_ANGLE, U1 APX803S-SA, U10 AMO091-12832BFG02-H14, U11 APX803S-SA, U12 AMO091-12832BFG02-H14, U13 APX803S-SA, U14 AMO091-12832BFG02-H14, U15 APX803S-SA, U16 AMO091-12832BFG02-H14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

Commit message: Repanelizes the design now that it has vertical Qwiic connectors
Parts:
- J1, J10, J11, J12, J13, J14, J15, J16, J17, J18, J19, J2, J20, J21, J22, J23, J24, J25, J26, J27, J28, J29, J3, J30, J31, J32, J33, J34, J35, J36, J37, J38, J39, J4, J40, J41, J42, J43, J44, J45, J46, J47, J48, J49, J5, J50, J51, J52, J53, J54, J55, J56, J57, J58, J59, J6, J60, J61, J62, J63, J64, J65, J66, J67, J68, J69, J7, J70, J71, J72, J8, J9: value QWIIC_RIGHT_ANGLE -> Vertical Qwiic Connector; device SparkFun-Connectors:JST04_1MM_RA -> SparkFun-Connectors:JST04_1MM_VERT
- turned J1 to 90 degrees
- turned J10 to 90 degrees
- turned J11 to 270 degrees
- turned J12 to 90 degrees
- turned J13 to 270 degrees
- turned J14 to 90 degrees
- turned J15 to 270 degrees
- turned J16 to 90 degrees
- turned J17 to 270 degrees
- turned J18 to 90 degrees
- turned J19 to 270 degrees
- turned J2 to 270 degrees
- turned J20 to 90 degrees
- turned J21 to 270 degrees
- turned J22 to 90 degrees
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Routing:
- net 3.3V34: track 46.2 -> 52.8 mm, vias 1 -> 3
- net 3.3V2: track 46.2 -> 52.8 mm, vias 1 -> 3
- net 3.3V10: track 46.2 -> 52.8 mm, vias 1 -> 3
- net 3.3V6: track 46.2 -> 52.8 mm, vias 1 -> 3
- net 3.3V32: track 46.2 -> 52.8 mm, vias 1 -> 3
- net 3.3V30: track 46.2 -> 52.8 mm, vias 1 -> 3
- net 3.3V26: track 46.2 -> 52.8 mm, vias 1 -> 3
- net 3.3V22: track 46.2 -> 52.8 mm, vias 1 -> 3
- net 3.3V8: track 46.2 -> 52.8 mm, vias 1 -> 3
- net 3.3V14: track 46.2 -> 52.8 mm, vias 1 -> 3
- net 3.3V33: track 46.2 -> 52.8 mm, vias 1 -> 3
- net 3.3V28: track 46.2 -> 52.8 mm, vias 1 -> 3
- net 3.3V24: track 46.2 -> 52.8 mm, vias 1 -> 3
- net 3.3V18: track 46.2 -> 52.8 mm, vias 1 -> 3
- net 3.3V20: track 46.2 -> 52.8 mm, vias 1 -> 3
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